File: audio_interface.kicad_pcb (KiCad board)
At the start: 2 copper layers, 26 parts, among them J1 AudioJack2, J2 XLR3_Ground, U1 OPA1655D, U2 OPA1655D, U3 OPA1655D

Commit message: implementing full adc and semi-microcontroller
Parts:
- added U4: PCM1860DBT, Package_SO:TSSOP-30_4.4x7.8mm_P0.5mm, F.Cu at (177.9, 110.3)
- added U5: STM32F401CDUx, Package_DFN_QFN:QFN-48-1EP_7x7mm_P0.5mm_EP5.6x5.6mm, F.Cu at (187.3, 110.2)
- RV1, RV2: footprint Potentiometer_THT:Potentiometer_Bourns_PTV09A-2_Single_Horizontal -> Potentiometer_THT:Potentiometer_Alps_RK09K_Single_Horizontal
Connections:
- net Net-(RV1-Pad3) renamed /MIC_AMP_OUT
- net Net-(RV2-Pad3) renamed /LINE_AMP_OUT

Commit message: wow... just wow...
Parts:
- removed U5: STM32F401CDUx, Package_DFN_QFN:QFN-48-1EP_7x7mm_P0.5mm_EP5.6x5.6mm
- added U6: STM32F401RBTx, Package_QFP:LQFP-64_10x10mm_P0.5mm, F.Cu at (201.2, 111.2)
Connections:
- U4 pad 10: Net-(U4-XI) -> unconnected-(U4-XI-Pad10)
- U4 pad 15: unconnected-(U4-SCKI-Pad15) -> /adc/MCK
- U4 pad 16: unconnected-(U4-LRCK-Pad16) -> /adc/I2S_WS
- U4 pad 17: unconnected-(U4-BCK-Pad17) -> /adc/I2S_CK
- U4 pad 18: unconnected-(U4-DOUT-Pad18) -> /adc/I2S_SD
- U4 pad 9: Net-(U4-XO) -> unconnected-(U4-XO-Pad9)
