File: power.kicad_sch (KiCad schematic)
At the start: 1 part, among them J3 USB_C_Receptacle_USB2.0_16P

Commit message: add schematic document
Connections:
- net at J3.A1 (GND), J3.A12 (GND), J3.B1 (GND)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: now also J3.SH (SHIELD)
- net at J3.A6 (D+): now also J3.B6 (D+)
- net at J3.A7 (D-): now also J3.B7 (D-)
Changed lines of the file:
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@@
 	(generator_version "10.0")
 	(paper "A4")
+	(wire
+		(pts
+			(xy 20.32 59.69) (xy 27.94 59.69)
+		)
+		(stroke
+			(width 0)
+			(type default)
+		)
+	)
+	(wire
+		(pts
+			(xy 43.18 34.29) (xy 43.18 36.83)
+		)
+		(stroke
+			(width 0)
+			(type default)
+		)
+	)
+	(wire
+		(pts
+			(xy 43.18 39.37) (xy 43.18 41.91)
+		)
+		(stroke
+			(width 0)
+			(type default)
+		)
+	)
 	(symbol
 		(lib_id "Connector:USB_C_Receptacle_USB2.0_16P")
